Commit message: New version with 2d laser and 3d in middle plate

File: turtlebot_description/robots/kobuki_hexagons1_astra_ust10lx_reactor_wrist.urdf.xacro (robot description, xacro)
@@ -4,5 +4,5 @@
     - Stacks    : hexagons
     - 3d Sensor : astra
-    - top_plate : urg04lx
+    - top_plate : reactor_wrist
 -->
 <robot name="turtlebot" xmlns:xacro="http://ros.org/wiki/xacro">
@@ -13,6 +13,9 @@
 	  <origin xyz="-0.086 0.008 0.094" rpy="0.0 0.0 0.0"/>
   </sensor_astra>
-  <sensor_hokuyo_urg04lx name="hokuyo" parent="plate_top_link" >
-		<origin xyz="0.137 0 0.0525" rpy="0 0 0" />
-  </sensor_hokuyo_urg04lx>
+  <sensor_hokuyo_ust10lx name="hokuyo" parent="plate_middle_link" >
+		<origin xyz="0.137 0 -0.0525" rpy="-3.14 0 0" />
+  </sensor_hokuyo_ust10lx>
+  <phantomx_reactor_wrist parent="plate_top_link" prefix="arm_">
+		<origin xyz="0.0 0.0 0.003" rpy="0.0 0.0 0.0"/>
+  </phantomx_reactor_wrist>
 </robot>

File: turtlebot_description/robots/kobuki_hexagons_astra_.urdf.xacro (robot description, xacro)
@@ -9,4 +9,6 @@
   <kobuki/>
   <stack_hexagons parent="base_link"/>
-  <sensor_astra parent="base_link"/>
+  <sensor_astra parent="plate_middle_link">
+	  <origin xyz="-0.086 0.008 0.094" rpy="0.0 0.0 0.0"/>
+  </sensor_astra>
 </robot>

File: turtlebot_description/robots/kobuki_hexagons_astra_reactor_no_wrist.urdf.xacro (robot description, xacro)
@@ -10,5 +10,7 @@
   <kobuki/>
   <stack_hexagons parent="base_link"/>
-  <sensor_astra parent="base_link"/>
+  <sensor_astra parent="plate_middle_link">
+	  <origin xyz="-0.086 0.008 0.094" rpy="0.0 0.0 0.0"/>
+  </sensor_astra>
   <phantomx_reactor_no_wrist parent="plate_top_link" prefix="arm_">
 		<origin xyz="0.0 0.0 0.003" rpy="0.0 0.0 0.0"/>

File: turtlebot_description/robots/kobuki_hexagons_astra_widowx.urdf.xacro (robot description, xacro)
@@ -10,5 +10,7 @@
   <kobuki/>
   <stack_hexagons parent="base_link"/>
-  <sensor_astra parent="base_link"/>
+  <sensor_astra parent="plate_middle_link">
+	  <origin xyz="-0.086 0.008 0.094" rpy="0.0 0.0 0.0"/>
+  </sensor_astra>
   <widowx_arm parent="plate_top_link" prefix="">
 		<origin xyz="0.045 0.0 0.003" rpy="0.0 0.0 0.0"/>

File: turtlebot_description/robots/kobuki_hexagons_no3d_notop.urdf.xacro (robot description, xacro)
@@ -3,6 +3,5 @@
     - Base      : kobuki
     - Stacks    : hexagons
-    - 3d Sensor : astra
-    - top_plate : urg04lx
+    - 3d Sensor : kinect
 -->
 <robot name="turtlebot" xmlns:xacro="http://ros.org/wiki/xacro">
@@ -10,9 +9,3 @@
   <kobuki/>
   <stack_hexagons parent="base_link"/>
-  <sensor_astra parent="plate_middle_link">
-	  <origin xyz="-0.086 0.008 0.094" rpy="0.0 0.0 0.0"/>
-  </sensor_astra>
-  <sensor_hokuyo_urg04lx name="hokuyo" parent="plate_top_link" >
-		<origin xyz="0.137 0 0.0525" rpy="0 0 0" />
-  </sensor_hokuyo_urg04lx>
 </robot>

File: turtlebot_description/urdf/sensors/astra.urdf.xacro (robot description, xacro)
@@ -11,8 +11,7 @@
   <xacro:property name="astra_dae_display_scale"   value="1.0" />
   <!-- Parameterised in part by the values in turtlebot_properties.urdf.xacro -->
-  <xacro:macro name="sensor_astra" params="parent">
+  <xacro:macro name="sensor_astra" params="parent *origin">
     <joint name="camera_rgb_joint" type="fixed">
-      <origin xyz="${astra_cam_px} ${astra_cam_py} ${astra_cam_pz}"
-              rpy="0 0 0"/>
+      <insert_block name="origin" />
       <parent link="${parent}"/>
       <child link="camera_rgb_frame" />

File: turtlebot_description/urdf/turtlebot_library.urdf.xacro (robot description, xacro)
@@ -13,4 +13,5 @@
   <xacro:include filename="$(find turtlebot_description)/urdf/stacks/circles.urdf.xacro"/>
   <xacro:include filename="$(find turtlebot_description)/urdf/stacks/hexagons.urdf.xacro"/>
+  <xacro:include filename="$(find turtlebot_description)/urdf/stacks/hexagons1.urdf.xacro"/>
   <!-- 3D Sensors -->
   <xacro:include filename="$(find turtlebot_description)/urdf/sensors/kinect.urdf.xacro"/>
@@ -21,4 +22,5 @@
   <xacro:include filename="$(find turtlebot_description)/urdf/sensors/rplidar.urdf.xacro"/>
   <xacro:include filename="$(find turtlebot_description)/urdf/sensors/hokuyo_urg04lx.urdf.xacro"/>
+  <xacro:include filename="$(find turtlebot_description)/urdf/sensors/hokuyo_ust10lx.urdf.xacro"/>
   <!-- Arms -->
   <xacro:include filename="$(find widowx_arm_description)/urdf/widowx.urdf.xacro"/>
