Commit message: moving urg position in model and adding launch file for urg lasers

File: turtlebot_description/robots/kobuki_hexagons_urg04lx_notop.urdf.xacro (robot description, xacro)
@@ -10,5 +10,5 @@
   <stack_hexagons parent="base_link"/>
   <sensor_hokuyo_urg04lx name="hokuyo" parent="plate_middle_link" >
-		<origin xyz="0.137 0 0.0525" rpy="0 0 0" />
+		<origin xyz="0.160 0 0.0525" rpy="0 0 0" />
   </sensor_hokuyo_urg04lx>
 </robot>

File: turtlebot_description/urdf/turtlebot_library.urdf.xacro (robot description, xacro)
@@ -21,7 +21,7 @@
   <xacro:include filename="$(find turtlebot_description)/urdf/sensors/rplidar.urdf.xacro"/>
   <xacro:include filename="$(find turtlebot_description)/urdf/sensors/hokuyo_urg04lx.urdf.xacro"/>
-  <!-- Arms -->
+  <!-- Arms >
   <xacro:include filename="$(find widowx_arm_description)/urdf/widowx.urdf.xacro"/>
   <xacro:include filename="$(find phantomx_reactor_arm_description)/urdf/phantomx_reactor_no_wrist.urdf.xacro"/>
-  <xacro:include filename="$(find phantomx_reactor_arm_description)/urdf/phantomx_reactor_wrist.urdf.xacro"/>
+  <xacro:include filename="$(find phantomx_reactor_arm_description)/urdf/phantomx_reactor_wrist.urdf.xacro"/-->
 </robot>
