Commit message: description: adding new combination of sensors: astra + rplidar 2

File: turtlebot_description/urdf/sensors/astra.urdf.xacro (robot description, xacro)
@@ -4,7 +4,7 @@
   <xacro:include filename="$(find turtlebot_description)/urdf/turtlebot_properties.urdf.xacro"/>
   <!-- Xacro properties -->
-  <xacro:property name="astra_cam_py" value="-0.0125"/>
+  <xacro:property name="astra_cam_py" value="0.025"/>
   <xacro:property name="astra_depth_rel_rgb_py" value="0.0250" />
-  <xacro:property name="astra_cam_rel_rgb_py"   value="-0.0125" />
+  <xacro:property name="astra_cam_rel_rgb_py"   value="0.0125" />
   <xacro:property name="astra_dae_display_scale"   value="1.0" />
   <!-- Parameterised in part by the values in turtlebot_properties.urdf.xacro -->

Commit message: kinetic-aidimme

File: turtlebot_description/urdf/sensors/astra.urdf.xacro (robot description, xacro)
@@ -4,5 +4,5 @@
   <xacro:include filename="$(find turtlebot_description)/urdf/turtlebot_properties.urdf.xacro"/>
   <!-- Xacro properties -->
-  <xacro:property name="astra_cam_py" value="0.025"/>
+  <!-- xacro:property name="astra_cam_py" value="0.025"/ -->
   <xacro:property name="astra_depth_rel_rgb_py" value="0.0250" />
   <xacro:property name="astra_cam_rel_rgb_py"   value="0.0125" />
