Commit message: First version of melodic

File: turtlebot_description/urdf/stacks/hexagons.urdf.xacro (robot description, xacro)
@@ -93,5 +93,5 @@
     </link>
   </xacro:macro>
-  <xacro:macro name="stack_3d_sensor_pole" params="parent number x_loc y_loc z_loc">
+  <xacro:macro name="stack_mid_plate_device_pole" params="parent number x_loc y_loc z_loc">
     <joint name="pole_kinect_${number}_joint" type="fixed">
       <origin xyz="${x_loc} ${y_loc} ${z_loc}" rpy="0 0 0"/>
@@ -193,6 +193,6 @@
     <stack_top_pole parent="${parent}" number="2" x_loc="-0.0381" y_loc= "0.1505" z_loc="0.2920"/>
     <stack_top_pole parent="${parent}" number="3" x_loc="-0.0381" y_loc="-0.1505" z_loc="0.2920"/>
-    <stack_3d_sensor_pole parent="${parent}" number="0" x_loc="-0.1024" y_loc= "0.098" z_loc="0.2372"/>
-    <stack_3d_sensor_pole parent="${parent}" number="1" x_loc="-0.1024" y_loc="-0.098" z_loc="0.2372"/>
+    <stack_mid_plate_device_pole parent="${parent}" number="0" x_loc="-0.1024" y_loc= "0.098" z_loc="0.2372"/>
+    <stack_mid_plate_device_pole parent="${parent}" number="1" x_loc="-0.1024" y_loc="-0.098" z_loc="0.2372"/>
     <joint name="plate_top_joint" type="fixed">
       <origin xyz="-0.01364 0.0  0.3966" rpy="0 0 0"/>

File: turtlebot_description/urdf/stacks/hexagons_upper.urdf.xacro (robot description, xacro)
@@ -94,5 +94,5 @@
     </link>
   </xacro:macro>
-  <xacro:macro name="stack_3d_sensor_pole" params="parent number x_loc y_loc z_loc">
+  <xacro:macro name="stack_mid_plate_device_pole" params="parent number x_loc y_loc z_loc">
     <joint name="pole_kinect_${number}_joint" type="fixed">
       <origin xyz="${x_loc} ${y_loc} ${z_loc+MIDDLE_PLATE_OFFSET}" rpy="0 0 0"/>
@@ -195,6 +195,6 @@
     <stack_top_pole parent="${parent}" number="2" x_loc="-0.0381" y_loc= "0.1505" z_loc="0.2920"/>
     <stack_top_pole parent="${parent}" number="3" x_loc="-0.0381" y_loc="-0.1505" z_loc="0.2920"/>
-    <stack_3d_sensor_pole parent="${parent}" number="0" x_loc="-0.1024" y_loc= "0.098" z_loc="0.2372"/>
-    <stack_3d_sensor_pole parent="${parent}" number="1" x_loc="-0.1024" y_loc="-0.098" z_loc="0.2372"/>
+    <stack_mid_plate_device_pole parent="${parent}" number="0" x_loc="-0.1024" y_loc= "0.098" z_loc="0.2372"/>
+    <stack_mid_plate_device_pole parent="${parent}" number="1" x_loc="-0.1024" y_loc="-0.098" z_loc="0.2372"/>
     <joint name="plate_top_joint" type="fixed">
       <origin xyz="-0.01364 0.0  ${0.3966+MIDDLE_PLATE_OFFSET}" rpy="0 0 0"/>
